Commit message: Allows one to parameterize every joint limit in the urdf.

File: ur_description/urdf/ur10.urdf.xacro (robot description, xacro)
@@ -55,5 +55,5 @@
     </inertial>
   </xacro:macro>
-  <xacro:macro name="ur10_robot" params="prefix joint_limited">
+  <xacro:macro name="ur10_robot" params="prefix j1_lwr_lmt j1_upr_lmt j2_lwr_lmt j2_upr_lmt j3_lwr_lmt j3_upr_lmt j4_lwr_lmt j4_upr_lmt j5_lwr_lmt j5_upr_lmt j6_lwr_lmt j6_upr_lmt">
     <link name="${prefix}base_link" >
       <visual>
@@ -79,10 +79,5 @@
       <origin xyz="0.0 0.0 ${shoulder_height}" rpy="0.0 0.0 0.0" />
       <axis xyz="0 0 1" />
-      <xacro:unless value="${joint_limited}">
-        <limit lower="${-2.0 * pi}" upper="${2.0 * pi}" effort="330.0" velocity="2.16"/>
-      </xacro:unless>
-      <xacro:if value="${joint_limited}">
-        <limit lower="${-pi}" upper="${pi}" effort="330.0" velocity="2.16"/>
-      </xacro:if>
+        <limit lower="${j1_lwr_lmt}" upper="${j1_upr_lmt}" effort="330.0" velocity="2.16"/>
       <dynamics damping="0.0" friction="0.0"/>
     </joint>
@@ -110,10 +105,5 @@
       <origin xyz="0.0 ${shoulder_offset} 0.0" rpy="0.0 ${pi / 2.0} 0.0" />
       <axis xyz="0 1 0" />
-      <xacro:unless value="${joint_limited}">
-        <limit lower="${-2.0 * pi}" upper="${2.0 * pi}" effort="330.0" velocity="2.16"/>
-      </xacro:unless>
-      <xacro:if value="${joint_limited}">
-        <limit lower="${-pi}" upper="${pi}" effort="330.0" velocity="2.16"/>
-      </xacro:if>
+        <limit lower="${j2_lwr_lmt}" upper="${j2_upr_lmt}" effort="330.0" velocity="2.16"/>
       <dynamics damping="0.0" friction="0.0"/>
     </joint>
@@ -141,10 +131,5 @@
       <origin xyz="0.0 ${elbow_offset} ${upper_arm_length}" rpy="0.0 0.0 0.0" />
       <axis xyz="0 1 0" />
-      <xacro:unless value="${joint_limited}">
-        <limit lower="${-2.0 * pi}" upper="${2.0 * pi}" effort="150.0" velocity="3.15"/>
-      </xacro:unless>
-      <xacro:if value="${joint_limited}">
-        <limit lower="${-pi}" upper="${pi}" effort="150.0" velocity="3.15"/>
-      </xacro:if>
+        <limit lower="${j3_lwr_lmt}" upper="${j3_upr_lmt}" effort="150.0" velocity="3.15"/>
       <dynamics damping="0.0" friction="0.0"/>
     </joint>
@@ -172,10 +157,5 @@
       <origin xyz="0.0 0.0 ${forearm_length}" rpy="0.0 ${pi / 2.0} 0.0" />
       <axis xyz="0 1 0" />
-      <xacro:unless value="${joint_limited}">
-        <limit lower="${-2.0 * pi}" upper="${2.0 * pi}" effort="54.0" velocity="3.2"/>
-      </xacro:unless>
-      <xacro:if value="${joint_limited}">
-        <limit lower="${-pi}" upper="${pi}" effort="54.0" velocity="3.2"/>
-      </xacro:if>
+        <limit lower="${j4_lwr_lmt}" upper="${j4_upr_lmt}" effort="54.0" velocity="3.2"/>
       <dynamics damping="0.0" friction="0.0"/>
     </joint>
@@ -203,10 +183,5 @@
       <origin xyz="0.0 ${wrist_1_length} 0.0" rpy="0.0 0.0 0.0" />
       <axis xyz="0 0 1" />
-      <xacro:unless value="${joint_limited}">
-        <limit lower="${-2.0 * pi}" upper="${2.0 * pi}" effort="54.0" velocity="3.2"/>
-      </xacro:unless>
-      <xacro:if value="${joint_limited}">
-        <limit lower="${-pi}" upper="${pi}" effort="54.0" velocity="3.2"/>
-      </xacro:if>
+        <limit lower="${j5_lwr_lmt}" upper="${j5_upr_lmt}" effort="54.0" velocity="3.2"/>
       <dynamics damping="0.0" friction="0.0"/>
     </joint>
@@ -234,10 +209,5 @@
       <origin xyz="0.0 0.0 ${wrist_2_length}" rpy="0.0 0.0 0.0" />
       <axis xyz="0 1 0" />
-      <xacro:unless value="${joint_limited}">
-        <limit lower="${-2.0 * pi}" upper="${2.0 * pi}" effort="54.0" velocity="3.2"/>
-      </xacro:unless>
-      <xacro:if value="${joint_limited}">
-        <limit lower="${-pi}" upper="${pi}" effort="54.0" velocity="3.2"/>
-      </xacro:if>
+        <limit lower="${j6_lwr_lmt}" upper="${j6_upr_lmt}" effort="54.0" velocity="3.2"/>
       <dynamics damping="0.0" friction="0.0"/>
     </joint>

File: ur_description/urdf/ur10_joint_limited_robot.urdf.xacro (robot description, xacro)
@@ -7,5 +7,12 @@
   <xacro:include filename="$(find ur_description)/urdf/ur10.urdf.xacro" />
   <!-- arm -->
-  <xacro:ur10_robot prefix="" joint_limited="true"/>
+  <xacro:ur10_robot prefix=""
+                    j1_lwr_lmt="${-pi}" j1_upr_lmt="${pi}"
+                    j2_lwr_lmt="${-pi}" j2_upr_lmt="${pi}"
+                    j3_lwr_lmt="${-pi}" j3_upr_lmt="${pi}"
+                    j4_lwr_lmt="${-pi}" j4_upr_lmt="${pi}"
+                    j5_lwr_lmt="${-pi}" j5_upr_lmt="${pi}"
+                    j6_lwr_lmt="${-pi}" j6_upr_lmt="${pi}"
+  />
   <link name="world" />
   <joint name="world_joint" type="fixed">

File: ur_description/urdf/ur10_robot.urdf.xacro (robot description, xacro)
@@ -7,5 +7,12 @@
   <xacro:include filename="$(find ur_description)/urdf/ur10.urdf.xacro" />
   <!-- arm -->
-  <xacro:ur10_robot prefix="" joint_limited="false"/>
+  <xacro:ur10_robot prefix=""
+                    j1_lwr_lmt="${-2.0*pi}" j1_upr_lmt="${2.0*pi}"
+                    j2_lwr_lmt="${-2.0*pi}" j2_upr_lmt="${2.0*pi}"
+                    j3_lwr_lmt="${-2.0*pi}" j3_upr_lmt="${2.0*pi}"
+                    j4_lwr_lmt="${-2.0*pi}" j4_upr_lmt="${2.0*pi}"
+                    j5_lwr_lmt="${-2.0*pi}" j5_upr_lmt="${2.0*pi}"
+                    j6_lwr_lmt="${-2.0*pi}" j6_upr_lmt="${2.0*pi}"
+  />
   <link name="world" />
   <joint name="world_joint" type="fixed">

File: ur_description/urdf/ur5.urdf.xacro (robot description, xacro)
@@ -70,5 +70,5 @@
     </inertial>
   </xacro:macro>
-  <xacro:macro name="ur5_robot" params="prefix joint_limited">
+  <xacro:macro name="ur5_robot" params="prefix j1_lwr_lmt j1_upr_lmt j2_lwr_lmt j2_upr_lmt j3_lwr_lmt j3_upr_lmt j4_lwr_lmt j4_upr_lmt j5_lwr_lmt j5_upr_lmt j6_lwr_lmt j6_upr_lmt">
     <link name="${prefix}base_link" >
       <visual>
@@ -93,10 +93,5 @@
       <origin xyz="0.0 0.0 ${shoulder_height}" rpy="0.0 0.0 0.0" />
       <axis xyz="0 0 1" />
-      <xacro:unless value="${joint_limited}">
-        <limit lower="${-2.0 * pi}" upper="${2.0 * pi}" effort="150.0" velocity="3.15"/>
-      </xacro:unless>
-      <xacro:if value="${joint_limited}">
-        <limit lower="${-pi}" upper="${pi}" effort="150.0" velocity="3.15"/>
-      </xacro:if>
+        <limit lower="${j1_lwr_lmt}" upper="${j1_upr_lmt}" effort="150.0" velocity="3.15"/>
       <dynamics damping="0.0" friction="0.0"/>
     </joint>
@@ -122,10 +117,5 @@
       <origin xyz="0.0 ${shoulder_offset} 0.0" rpy="0.0 ${pi / 2.0} 0.0" />
       <axis xyz="0 1 0" />
-      <xacro:unless value="${joint_limited}">
-        <limit lower="${-2.0 * pi}" upper="${2.0 * pi}" effort="150.0" velocity="3.15"/>
-      </xacro:unless>
-      <xacro:if value="${joint_limited}">
-        <limit lower="${-pi}" upper="${pi}" effort="150.0" velocity="3.15"/>
-      </xacro:if>
+        <limit lower="${j2_lwr_lmt}" upper="${j2_upr_lmt}" effort="150.0" velocity="3.15"/>
       <dynamics damping="0.0" friction="0.0"/>
     </joint>
@@ -152,10 +142,5 @@
       <origin xyz="0.0 ${elbow_offset} ${upper_arm_length}" rpy="0.0 0.0 0.0" />
       <axis xyz="0 1 0" />
-      <xacro:unless value="${joint_limited}">
-        <limit lower="${-2.0 * pi}" upper="${2.0 * pi}" effort="150.0" velocity="3.15"/>
-      </xacro:unless>
-      <xacro:if value="${joint_limited}">
-        <limit lower="${-pi}" upper="${pi}" effort="150.0" velocity="3.15"/>
-      </xacro:if>
+        <limit lower="${j3_lwr_lmt}" upper="${j3_upr_lmt}" effort="150.0" velocity="3.15"/>
       <dynamics damping="0.0" friction="0.0"/>
     </joint>
@@ -181,10 +166,5 @@
       <origin xyz="0.0 0.0 ${forearm_length}" rpy="0.0 ${pi / 2.0} 0.0" />
       <axis xyz="0 1 0" />
-      <xacro:unless value="${joint_limited}">
-        <limit lower="${-2.0 * pi}" upper="${2.0 * pi}" effort="28.0" velocity="3.2"/>
-      </xacro:unless>
-      <xacro:if value="${joint_limited}">
-        <limit lower="${-pi}" upper="${pi}" effort="28.0" velocity="3.2"/>
-      </xacro:if>
+        <limit lower="${j4_lwr_lmt}" upper="${j4_upr_lmt}" effort="28.0" velocity="3.2"/>
       <dynamics damping="0.0" friction="0.0"/>
     </joint>
@@ -211,10 +191,5 @@
       <origin xyz="0.0 ${wrist_1_length} 0.0" rpy="0.0 0.0 0.0" />
       <axis xyz="0 0 1" />
-      <xacro:unless value="${joint_limited}">
-        <limit lower="${-2.0 * pi}" upper="${2.0 * pi}" effort="28.0" velocity="3.2"/>
-      </xacro:unless>
-      <xacro:if value="${joint_limited}">
-        <limit lower="${-pi}" upper="${pi}" effort="28.0" velocity="3.2"/>
-      </xacro:if>
+        <limit lower="${j5_lwr_lmt}" upper="${j5_upr_lmt}" effort="28.0" velocity="3.2"/>
       <dynamics damping="0.0" friction="0.0"/>
     </joint>
@@ -241,10 +216,5 @@
       <origin xyz="0.0 0.0 ${wrist_2_length}" rpy="0.0 0.0 0.0" />
       <axis xyz="0 1 0" />
-      <xacro:unless value="${joint_limited}">
-        <limit lower="${-2.0 * pi}" upper="${2.0 * pi}" effort="28.0" velocity="3.2"/>
-      </xacro:unless>
-      <xacro:if value="${joint_limited}">
-        <limit lower="${-pi}" upper="${pi}" effort="28.0" velocity="3.2"/>
-      </xacro:if>
+        <limit lower="${j6_lwr_lmt}" upper="${j6_upr_lmt}" effort="28.0" velocity="3.2"/>
       <dynamics damping="0.0" friction="0.0"/>
     </joint>

File: ur_description/urdf/ur5_joint_limited_robot.urdf.xacro (robot description, xacro)
@@ -7,5 +7,12 @@
   <xacro:include filename="$(find ur_description)/urdf/ur5.urdf.xacro" />
   <!-- arm -->
-  <xacro:ur5_robot prefix="" joint_limited="true"/>
+  <xacro:ur5_robot prefix=""
+                   j1_lwr_lmt="${-pi}" j1_upr_lmt="${pi}"
+                   j2_lwr_lmt="${-pi}" j2_upr_lmt="${pi}"
+                   j3_lwr_lmt="${-pi}" j3_upr_lmt="${pi}"
+                   j4_lwr_lmt="${-pi}" j4_upr_lmt="${pi}"
+                   j5_lwr_lmt="${-pi}" j5_upr_lmt="${pi}"
+                   j6_lwr_lmt="${-pi}" j6_upr_lmt="${pi}"
+  />
   <link name="world" />
   <joint name="world_joint" type="fixed">

File: ur_description/urdf/ur5_robot.urdf.xacro (robot description, xacro)
@@ -7,5 +7,12 @@
   <xacro:include filename="$(find ur_description)/urdf/ur5.urdf.xacro" />
   <!-- arm -->
-  <xacro:ur5_robot prefix="" joint_limited="false"/>
+  <xacro:ur5_robot prefix=""
+                   j1_lwr_lmt="${-2.0*pi}" j1_upr_lmt="${2.0*pi}"
+                   j2_lwr_lmt="${-2.0*pi}" j2_upr_lmt="${2.0*pi}"
+                   j3_lwr_lmt="${-2.0*pi}" j3_upr_lmt="${2.0*pi}"
+                   j4_lwr_lmt="${-2.0*pi}" j4_upr_lmt="${2.0*pi}"
+                   j5_lwr_lmt="${-2.0*pi}" j5_upr_lmt="${2.0*pi}"
+                   j6_lwr_lmt="${-2.0*pi}" j6_upr_lmt="${2.0*pi}"
+  />
   <link name="world" />
   <joint name="world_joint" type="fixed">
