Commit message: Updating URDFs to also parameterize joint velocity limits.

File: ur_description/urdf/ur10.urdf.xacro (robot description, xacro)
@@ -55,5 +55,5 @@
     </inertial>
   </xacro:macro>
-  <xacro:macro name="ur10_robot" params="prefix j1_lwr_lmt j1_upr_lmt j2_lwr_lmt j2_upr_lmt j3_lwr_lmt j3_upr_lmt j4_lwr_lmt j4_upr_lmt j5_lwr_lmt j5_upr_lmt j6_lwr_lmt j6_upr_lmt">
+  <xacro:macro name="ur10_robot" params="prefix j1_lwr_lmt j1_upr_lmt j1_vel_lmt j2_lwr_lmt j2_upr_lmt j2_vel_lmt j3_lwr_lmt j3_upr_lmt j3_vel_lmt j4_lwr_lmt j4_upr_lmt j4_vel_lmt j5_lwr_lmt j5_upr_lmt j5_vel_lmt j6_lwr_lmt j6_upr_lmt j6_vel_lmt">
     <link name="${prefix}base_link" >
       <visual>
@@ -79,5 +79,5 @@
       <origin xyz="0.0 0.0 ${shoulder_height}" rpy="0.0 0.0 0.0" />
       <axis xyz="0 0 1" />
-        <limit lower="${j1_lwr_lmt}" upper="${j1_upr_lmt}" effort="330.0" velocity="2.16"/>
+        <limit lower="${j1_lwr_lmt}" upper="${j1_upr_lmt}" effort="330.0" velocity="${j1_vel_lmt}"/>
       <dynamics damping="0.0" friction="0.0"/>
     </joint>
@@ -105,5 +105,5 @@
       <origin xyz="0.0 ${shoulder_offset} 0.0" rpy="0.0 ${pi / 2.0} 0.0" />
       <axis xyz="0 1 0" />
-        <limit lower="${j2_lwr_lmt}" upper="${j2_upr_lmt}" effort="330.0" velocity="2.16"/>
+        <limit lower="${j2_lwr_lmt}" upper="${j2_upr_lmt}" effort="330.0" velocity="${j2_vel_lmt}"/>
       <dynamics damping="0.0" friction="0.0"/>
     </joint>
@@ -131,5 +131,5 @@
       <origin xyz="0.0 ${elbow_offset} ${upper_arm_length}" rpy="0.0 0.0 0.0" />
       <axis xyz="0 1 0" />
-        <limit lower="${j3_lwr_lmt}" upper="${j3_upr_lmt}" effort="150.0" velocity="3.15"/>
+        <limit lower="${j3_lwr_lmt}" upper="${j3_upr_lmt}" effort="150.0" velocity="${j3_vel_lmt}"/>
       <dynamics damping="0.0" friction="0.0"/>
     </joint>
@@ -157,5 +157,5 @@
       <origin xyz="0.0 0.0 ${forearm_length}" rpy="0.0 ${pi / 2.0} 0.0" />
       <axis xyz="0 1 0" />
-        <limit lower="${j4_lwr_lmt}" upper="${j4_upr_lmt}" effort="54.0" velocity="3.2"/>
+        <limit lower="${j4_lwr_lmt}" upper="${j4_upr_lmt}" effort="54.0" velocity="${j4_vel_lmt}"/>
       <dynamics damping="0.0" friction="0.0"/>
     </joint>
@@ -183,5 +183,5 @@
       <origin xyz="0.0 ${wrist_1_length} 0.0" rpy="0.0 0.0 0.0" />
       <axis xyz="0 0 1" />
-        <limit lower="${j5_lwr_lmt}" upper="${j5_upr_lmt}" effort="54.0" velocity="3.2"/>
+        <limit lower="${j5_lwr_lmt}" upper="${j5_upr_lmt}" effort="54.0" velocity="${j5_vel_lmt}"/>
       <dynamics damping="0.0" friction="0.0"/>
     </joint>
@@ -209,5 +209,5 @@
       <origin xyz="0.0 0.0 ${wrist_2_length}" rpy="0.0 0.0 0.0" />
       <axis xyz="0 1 0" />
-        <limit lower="${j6_lwr_lmt}" upper="${j6_upr_lmt}" effort="54.0" velocity="3.2"/>
+        <limit lower="${j6_lwr_lmt}" upper="${j6_upr_lmt}" effort="54.0" velocity="${j6_vel_lmt}"/>
       <dynamics damping="0.0" friction="0.0"/>
     </joint>

File: ur_description/urdf/ur10_joint_limited_robot.urdf (robot description, URDF)
Before this commit: robot ur10, 9 links, 8 joints
Joints:
- joint elbow_joint: axis 0.0 1.0 0.0 -> 0 1 0
- joint shoulder_lift_joint: axis 0.0 1.0 0.0 -> 0 1 0
- joint shoulder_pan_joint: axis 0.0 0.0 1.0 -> 0 0 1
- joint wrist_1_joint: axis 0.0 1.0 0.0 -> 0 1 0
- joint wrist_2_joint: axis 0.0 0.0 1.0 -> 0 0 1
- joint wrist_3_joint: axis 0.0 1.0 0.0 -> 0 1 0

File: ur_description/urdf/ur10_joint_limited_robot.urdf.xacro (robot description, xacro)
@@ -8,10 +8,10 @@
   <!-- arm -->
   <xacro:ur10_robot prefix=""
-                    j1_lwr_lmt="${-pi}" j1_upr_lmt="${pi}"
-                    j2_lwr_lmt="${-pi}" j2_upr_lmt="${pi}"
-                    j3_lwr_lmt="${-pi}" j3_upr_lmt="${pi}"
-                    j4_lwr_lmt="${-pi}" j4_upr_lmt="${pi}"
-                    j5_lwr_lmt="${-pi}" j5_upr_lmt="${pi}"
-                    j6_lwr_lmt="${-pi}" j6_upr_lmt="${pi}"
+                    j1_lwr_lmt="${-pi}" j1_upr_lmt="${pi}" j1_vel_lmt="2.16"
+                    j2_lwr_lmt="${-pi}" j2_upr_lmt="${pi}" j2_vel_lmt="2.16"
+                    j3_lwr_lmt="${-pi}" j3_upr_lmt="${pi}" j3_vel_lmt="3.15"
+                    j4_lwr_lmt="${-pi}" j4_upr_lmt="${pi}" j4_vel_lmt="3.2"
+                    j5_lwr_lmt="${-pi}" j5_upr_lmt="${pi}" j5_vel_lmt="3.2"
+                    j6_lwr_lmt="${-pi}" j6_upr_lmt="${pi}" j6_vel_lmt="3.2"
   />
   <link name="world" />

File: ur_description/urdf/ur10_robot.urdf (robot description, URDF)
Before this commit: robot ur10, 9 links, 8 joints
Joints:
- joint elbow_joint: axis 0.0 1.0 0.0 -> 0 1 0
- joint shoulder_lift_joint: axis 0.0 1.0 0.0 -> 0 1 0
- joint shoulder_pan_joint: axis 0.0 0.0 1.0 -> 0 0 1
- joint wrist_1_joint: axis 0.0 1.0 0.0 -> 0 1 0
- joint wrist_2_joint: axis 0.0 0.0 1.0 -> 0 0 1
- joint wrist_3_joint: axis 0.0 1.0 0.0 -> 0 1 0

File: ur_description/urdf/ur10_robot.urdf.xacro (robot description, xacro)
@@ -8,10 +8,10 @@
   <!-- arm -->
   <xacro:ur10_robot prefix=""
-                    j1_lwr_lmt="${-2.0*pi}" j1_upr_lmt="${2.0*pi}"
-                    j2_lwr_lmt="${-2.0*pi}" j2_upr_lmt="${2.0*pi}"
-                    j3_lwr_lmt="${-2.0*pi}" j3_upr_lmt="${2.0*pi}"
-                    j4_lwr_lmt="${-2.0*pi}" j4_upr_lmt="${2.0*pi}"
-                    j5_lwr_lmt="${-2.0*pi}" j5_upr_lmt="${2.0*pi}"
-                    j6_lwr_lmt="${-2.0*pi}" j6_upr_lmt="${2.0*pi}"
+                    j1_lwr_lmt="${-2.0*pi}" j1_upr_lmt="${2.0*pi}" j1_vel_lmt="2.16"
+                    j2_lwr_lmt="${-2.0*pi}" j2_upr_lmt="${2.0*pi}" j2_vel_lmt="2.16"
+                    j3_lwr_lmt="${-2.0*pi}" j3_upr_lmt="${2.0*pi}" j3_vel_lmt="3.15"
+                    j4_lwr_lmt="${-2.0*pi}" j4_upr_lmt="${2.0*pi}" j4_vel_lmt="3.2"
+                    j5_lwr_lmt="${-2.0*pi}" j5_upr_lmt="${2.0*pi}" j5_vel_lmt="3.2"
+                    j6_lwr_lmt="${-2.0*pi}" j6_upr_lmt="${2.0*pi}" j6_vel_lmt="3.2"
   />
   <link name="world" />

File: ur_description/urdf/ur5.urdf.xacro (robot description, xacro)
@@ -70,5 +70,5 @@
     </inertial>
   </xacro:macro>
-  <xacro:macro name="ur5_robot" params="prefix j1_lwr_lmt j1_upr_lmt j2_lwr_lmt j2_upr_lmt j3_lwr_lmt j3_upr_lmt j4_lwr_lmt j4_upr_lmt j5_lwr_lmt j5_upr_lmt j6_lwr_lmt j6_upr_lmt">
+  <xacro:macro name="ur5_robot" params="prefix j1_lwr_lmt j1_upr_lmt j1_vel_lmt j2_lwr_lmt j2_upr_lmt j2_vel_lmt j3_lwr_lmt j3_upr_lmt j3_vel_lmt j4_lwr_lmt j4_upr_lmt j4_vel_lmt j5_lwr_lmt j5_upr_lmt j5_vel_lmt j6_lwr_lmt j6_upr_lmt j6_vel_lmt">
     <link name="${prefix}base_link" >
       <visual>
@@ -93,5 +93,5 @@
       <origin xyz="0.0 0.0 ${shoulder_height}" rpy="0.0 0.0 0.0" />
       <axis xyz="0 0 1" />
-        <limit lower="${j1_lwr_lmt}" upper="${j1_upr_lmt}" effort="150.0" velocity="3.15"/>
+        <limit lower="${j1_lwr_lmt}" upper="${j1_upr_lmt}" effort="150.0" velocity="${j1_vel_lmt}"/>
       <dynamics damping="0.0" friction="0.0"/>
     </joint>
@@ -117,5 +117,5 @@
       <origin xyz="0.0 ${shoulder_offset} 0.0" rpy="0.0 ${pi / 2.0} 0.0" />
       <axis xyz="0 1 0" />
-        <limit lower="${j2_lwr_lmt}" upper="${j2_upr_lmt}" effort="150.0" velocity="3.15"/>
+        <limit lower="${j2_lwr_lmt}" upper="${j2_upr_lmt}" effort="150.0" velocity="${j2_vel_lmt}"/>
       <dynamics damping="0.0" friction="0.0"/>
     </joint>
@@ -142,5 +142,5 @@
       <origin xyz="0.0 ${elbow_offset} ${upper_arm_length}" rpy="0.0 0.0 0.0" />
       <axis xyz="0 1 0" />
-        <limit lower="${j3_lwr_lmt}" upper="${j3_upr_lmt}" effort="150.0" velocity="3.15"/>
+        <limit lower="${j3_lwr_lmt}" upper="${j3_upr_lmt}" effort="150.0" velocity="${j3_vel_lmt}"/>
       <dynamics damping="0.0" friction="0.0"/>
     </joint>
@@ -166,5 +166,5 @@
       <origin xyz="0.0 0.0 ${forearm_length}" rpy="0.0 ${pi / 2.0} 0.0" />
       <axis xyz="0 1 0" />
-        <limit lower="${j4_lwr_lmt}" upper="${j4_upr_lmt}" effort="28.0" velocity="3.2"/>
+        <limit lower="${j4_lwr_lmt}" upper="${j4_upr_lmt}" effort="28.0" velocity="${j4_vel_lmt}"/>
       <dynamics damping="0.0" friction="0.0"/>
     </joint>
@@ -191,5 +191,5 @@
       <origin xyz="0.0 ${wrist_1_length} 0.0" rpy="0.0 0.0 0.0" />
       <axis xyz="0 0 1" />
-        <limit lower="${j5_lwr_lmt}" upper="${j5_upr_lmt}" effort="28.0" velocity="3.2"/>
+        <limit lower="${j5_lwr_lmt}" upper="${j5_upr_lmt}" effort="28.0" velocity="${j5_vel_lmt}"/>
       <dynamics damping="0.0" friction="0.0"/>
     </joint>
@@ -216,5 +216,5 @@
       <origin xyz="0.0 0.0 ${wrist_2_length}" rpy="0.0 0.0 0.0" />
       <axis xyz="0 1 0" />
-        <limit lower="${j6_lwr_lmt}" upper="${j6_upr_lmt}" effort="28.0" velocity="3.2"/>
+        <limit lower="${j6_lwr_lmt}" upper="${j6_upr_lmt}" effort="28.0" velocity="${j6_vel_lmt}"/>
       <dynamics damping="0.0" friction="0.0"/>
     </joint>

File: ur_description/urdf/ur5_joint_limited_robot.urdf (robot description, URDF)
Before this commit: robot ur5, 8 links, 7 joints
Links:
- added link world
Joints:
- added joint world_joint: type fixed, parent world, child base_link, origin xyz=0.0 0.0 0.0 rpy=0.0 0.0 0.0
- joint elbow_joint: limit lower=-3.14159265 upper=3.14159265 effort=150.0 velocity=3.14159265 -> lower=-3.14159265 upper=3.14159265 effort=150.0 velocity=3.15
- joint shoulder_lift_joint: limit lower=-3.14159265 upper=3.14159265 effort=150.0 velocity=3.14159265 -> lower=-3.14159265 upper=3.14159265 effort=150.0 velocity=3.15
- joint shoulder_pan_joint: limit lower=-3.14159265 upper=3.14159265 effort=150.0 velocity=3.14159265 -> lower=-3.14159265 upper=3.14159265 effort=150.0 velocity=3.15
- joint wrist_1_joint: limit lower=-3.14159265 upper=0.7853981625 effort=28.0 velocity=3.14159265 -> lower=-3.14159265 upper=3.14159265 effort=28.0 velocity=3.2
- joint wrist_2_joint: limit lower=-3.14159265 upper=3.14159265 effort=28.0 velocity=3.14159265 -> lower=-3.14159265 upper=3.14159265 effort=28.0 velocity=3.2
- joint wrist_3_joint: limit lower=-3.14159265 upper=3.14159265 effort=28.0 velocity=3.14159265 -> lower=-3.14159265 upper=3.14159265 effort=28.0 velocity=3.2

File: ur_description/urdf/ur5_joint_limited_robot.urdf.xacro (robot description, xacro)
@@ -8,10 +8,10 @@
   <!-- arm -->
   <xacro:ur5_robot prefix=""
-                   j1_lwr_lmt="${-pi}" j1_upr_lmt="${pi}"
-                   j2_lwr_lmt="${-pi}" j2_upr_lmt="${pi}"
-                   j3_lwr_lmt="${-pi}" j3_upr_lmt="${pi}"
-                   j4_lwr_lmt="${-pi}" j4_upr_lmt="${pi}"
-                   j5_lwr_lmt="${-pi}" j5_upr_lmt="${pi}"
-                   j6_lwr_lmt="${-pi}" j6_upr_lmt="${pi}"
+                    j1_lwr_lmt="${-pi}" j1_upr_lmt="${pi}" j1_vel_lmt="3.15"
+                    j2_lwr_lmt="${-pi}" j2_upr_lmt="${pi}" j2_vel_lmt="3.15"
+                    j3_lwr_lmt="${-pi}" j3_upr_lmt="${pi}" j3_vel_lmt="3.15"
+                    j4_lwr_lmt="${-pi}" j4_upr_lmt="${pi}" j4_vel_lmt="3.2"
+                    j5_lwr_lmt="${-pi}" j5_upr_lmt="${pi}" j5_vel_lmt="3.2"
+                    j6_lwr_lmt="${-pi}" j6_upr_lmt="${pi}" j6_vel_lmt="3.2"
   />
   <link name="world" />

File: ur_description/urdf/ur5_robot.urdf (robot description, URDF)
Before this commit: robot ur5, 8 links, 7 joints
Links:
- added link world
Joints:
- added joint world_joint: type fixed, parent world, child base_link, origin xyz=0.0 0.0 0.0 rpy=0.0 0.0 0.0
- joint elbow_joint: limit lower=-6.2831853 upper=6.2831853 effort=150.0 velocity=3.14159265 -> lower=-6.2831853 upper=6.2831853 effort=150.0 velocity=3.15
- joint shoulder_lift_joint: limit lower=-6.2831853 upper=6.2831853 effort=150.0 velocity=3.14159265 -> lower=-6.2831853 upper=6.2831853 effort=150.0 velocity=3.15
- joint shoulder_pan_joint: limit lower=-6.2831853 upper=6.2831853 effort=150.0 velocity=3.14159265 -> lower=-6.2831853 upper=6.2831853 effort=150.0 velocity=3.15
- joint wrist_1_joint: limit lower=-3.14159265 upper=0.7853981625 effort=28.0 velocity=3.14159265 -> lower=-6.2831853 upper=6.2831853 effort=28.0 velocity=3.2
- joint wrist_2_joint: limit lower=-3.14159265 upper=3.14159265 effort=28.0 velocity=3.14159265 -> lower=-6.2831853 upper=6.2831853 effort=28.0 velocity=3.2
- joint wrist_3_joint: limit lower=-3.14159265 upper=3.14159265 effort=28.0 velocity=3.14159265 -> lower=-6.2831853 upper=6.2831853 effort=28.0 velocity=3.2

File: ur_description/urdf/ur5_robot.urdf.xacro (robot description, xacro)
@@ -8,10 +8,10 @@
   <!-- arm -->
   <xacro:ur5_robot prefix=""
-                   j1_lwr_lmt="${-2.0*pi}" j1_upr_lmt="${2.0*pi}"
-                   j2_lwr_lmt="${-2.0*pi}" j2_upr_lmt="${2.0*pi}"
-                   j3_lwr_lmt="${-2.0*pi}" j3_upr_lmt="${2.0*pi}"
-                   j4_lwr_lmt="${-2.0*pi}" j4_upr_lmt="${2.0*pi}"
-                   j5_lwr_lmt="${-2.0*pi}" j5_upr_lmt="${2.0*pi}"
-                   j6_lwr_lmt="${-2.0*pi}" j6_upr_lmt="${2.0*pi}"
+                    j1_lwr_lmt="${-2.0*pi}" j1_upr_lmt="${2.0*pi}" j1_vel_lmt="3.15"
+                    j2_lwr_lmt="${-2.0*pi}" j2_upr_lmt="${2.0*pi}" j2_vel_lmt="3.15"
+                    j3_lwr_lmt="${-2.0*pi}" j3_upr_lmt="${2.0*pi}" j3_vel_lmt="3.15"
+                    j4_lwr_lmt="${-2.0*pi}" j4_upr_lmt="${2.0*pi}" j4_vel_lmt="3.2"
+                    j5_lwr_lmt="${-2.0*pi}" j5_upr_lmt="${2.0*pi}" j5_vel_lmt="3.2"
+                    j6_lwr_lmt="${-2.0*pi}" j6_upr_lmt="${2.0*pi}" j6_vel_lmt="3.2"
   />
   <link name="world" />

Commit message: Adding option to enable cylinders for collision model.

File: ur_description/urdf/ur10.urdf.xacro (robot description, xacro)
@@ -55,5 +55,5 @@
     </inertial>
   </xacro:macro>
-  <xacro:macro name="ur10_robot" params="prefix j1_lwr_lmt j1_upr_lmt j1_vel_lmt j2_lwr_lmt j2_upr_lmt j2_vel_lmt j3_lwr_lmt j3_upr_lmt j3_vel_lmt j4_lwr_lmt j4_upr_lmt j4_vel_lmt j5_lwr_lmt j5_upr_lmt j5_vel_lmt j6_lwr_lmt j6_upr_lmt j6_vel_lmt">
+  <xacro:macro name="ur10_robot" params="prefix cylinders_collision j1_lwr_lmt j1_upr_lmt j1_vel_lmt j2_lwr_lmt j2_upr_lmt j2_vel_lmt j3_lwr_lmt j3_upr_lmt j3_vel_lmt j4_lwr_lmt j4_upr_lmt j4_vel_lmt j5_lwr_lmt j5_upr_lmt j5_vel_lmt j6_lwr_lmt j6_upr_lmt j6_vel_lmt">
     <link name="${prefix}base_link" >
       <visual>
@@ -65,8 +65,16 @@
       </visual>
       <collision>
-        <geometry>
-          <mesh filename="package://ur_description/meshes/ur10/collision/Base.dae" scale="${scale}"/>
-        </geometry>
-        <origin xyz="0.0 0.0 0.0" rpy="${pi / 2.0} 0.0 0.0" />
+        <xacro:if value="${cylinders_collision}">
+          <geometry>
+            <cylinder length="0.04" radius="0.10" />
+          </geometry>
+        <origin xyz="0.0 0.0 0.02" rpy="0.0 0.0 0.0" />
+        </xacro:if>
+        <xacro:unless value="${cylinders_collision}">
+          <geometry>
+            <mesh filename="package://ur_description/meshes/ur10/collision/Base.dae" scale="${scale}"/>
+          </geometry>
+          <origin xyz="0.0 0.0 0.0" rpy="${pi / 2.0} 0.0 0.0" />
+        </xacro:unless>
       </collision>
       <xacro:cylinder_inertial radius="0.075" length="0.038" mass="${base_mass}">
@@ -91,8 +99,16 @@
       </visual>
       <collision>
-        <geometry>
-          <mesh filename="package://ur_description/meshes/ur10/collision/Shoulder.dae" scale="${scale}"/>
-        </geometry>
-        <origin rpy="${pi / 2.0} 0.0 0.0" xyz="0.0 0.0 -0.127"/>   <!-- -0.127 ????  -->
+        <xacro:if value="${cylinders_collision}">
+          <geometry>
+            <cylinder length="0.171" radius="0.08" />
+          </geometry>
+          <origin xyz="0.0 0.0 0.0" rpy="0.0 0.0 0.0" />
+        </xacro:if>
+        <xacro:unless value="${cylinders_collision}">
+          <geometry>
+            <mesh filename="package://ur_description/meshes/ur10/collision/Shoulder.dae" scale="${scale}"/>
+          </geometry>
+          <origin rpy="${pi / 2.0} 0.0 0.0" xyz="0.0 0.0 -0.127"/>   <!-- -0.127 ????  -->
+        </xacro:unless>
       </collision>
       <xacro:cylinder_inertial radius="0.075" length="0.178" mass="${shoulder_mass}">
@@ -117,8 +133,16 @@
       </visual>
       <collision>
-        <geometry>
-          <mesh filename="package://ur_description/meshes/ur10/collision/UpperArm.dae" scale="${scale}"/>
-        </geometry>
-        <origin xyz="0.0 -0.221 -0.127" rpy="${pi / 2.0} 0.0 0.0" />  <!-- new offset-->
+        <xacro:if value="${cylinders_collision}">
+          <geometry>
+            <cylinder length="${-ur10_a2+0.15}" radius="0.058" />
+          </geometry>
+          <origin xyz="0.0 -0.042 ${(-ur10_a2+0.15)/2-0.08}" rpy="0.0 0.0 0.0" />
+        </xacro:if>
+        <xacro:unless value="${cylinders_collision}">
+          <geometry>
+            <mesh filename="package://ur_description/meshes/ur10/collision/UpperArm.dae" scale="${scale}"/>
+          </geometry>
+          <origin xyz="0.0 -0.221 -0.127" rpy="${pi / 2.0} 0.0 0.0" />  <!-- new offset-->
+        </xacro:unless>
       </collision>
       <xacro:cylinder_inertial radius="0.075" length="${-ur10_a2}" mass="${upper_arm_mass}">
@@ -143,8 +167,16 @@
       </visual>
       <collision>
-        <geometry>
-          <mesh filename="package://ur_description/meshes/ur10/collision/Forearm.dae" scale="${scale}"/>
-        </geometry>
-        <origin xyz="0.0 -0.049 -0.739" rpy="${pi / 2.0} 0.0 0.0" />  <!-- new offset -->
+        <xacro:if value="${cylinders_collision}">
+          <geometry>
+            <cylinder length="${(-ur10_a3+0.05)}" radius="0.048" />
+          </geometry>
+          <origin xyz="0.0 0.0 ${(-ur10_a3+0.05)/2-0.06}" rpy="0.0 0.0 0.0" />
+        </xacro:if>
+        <xacro:unless value="${cylinders_collision}">
+          <geometry>
+            <mesh filename="package://ur_description/meshes/ur10/collision/Forearm.dae" scale="${scale}"/>
+          </geometry>
+          <origin xyz="0.0 -0.049 -0.739" rpy="${pi / 2.0} 0.0 0.0" />  <!-- new offset -->
+        </xacro:unless>
       </collision>
       <xacro:cylinder_inertial radius="0.075" length="${-ur10_a3}" mass="${forearm_mass}">
@@ -169,8 +201,16 @@
       </visual>
       <collision>
-        <geometry>
-          <mesh filename="package://ur_description/meshes/ur10/collision/Wrist1.dae" scale="${scale}"/>
-        </geometry>
-        <origin xyz="0.0 -0.049 -1.312" rpy="${pi / 2.0} 0 0.0" />  <!-- new offset -->
+        <xacro:if value="${cylinders_collision}">
+          <geometry>
+            <cylinder length="0.12" radius="0.047" />
+          </geometry>
+          <origin xyz="0.0 0.01 0.0" rpy="${pi/2} 0.0 0.0" />
+        </xacro:if>
+        <xacro:unless value="${cylinders_collision}">
+          <geometry>
+            <mesh filename="package://ur_description/meshes/ur10/collision/Wrist1.dae" scale="${scale}"/>
+          </geometry>
+          <origin xyz="0.0 -0.049 -1.312" rpy="${pi / 2.0} 0 0.0" />  <!-- new offset -->
+        </xacro:unless>
       </collision>
       <xacro:cylinder_inertial radius="0.075" length="0.12" mass="${wrist_1_mass}">
@@ -195,8 +235,16 @@
       </visual>
       <collision>
-        <geometry>
-          <mesh filename="package://ur_description/meshes/ur10/collision/Wrist2.dae" scale="${scale}"/>
-        </geometry>
-        <origin xyz="0.0 -0.164 -1.312" rpy="${pi / 2.0} 0.0 0.0" />  <!-- new offset -->
+        <xacro:if value="${cylinders_collision}">
+          <geometry>
+            <cylinder length="0.18" radius="0.046" />
+          </geometry>
+          <origin xyz="0.0 0.0 0.032" rpy="0.0 0.0 0.0" />
+        </xacro:if>
+        <xacro:unless value="${cylinders_collision}">
+          <geometry>
+            <mesh filename="package://ur_description/meshes/ur10/collision/Wrist2.dae" scale="${scale}"/>
+          </geometry>
+          <origin xyz="0.0 -0.164 -1.312" rpy="${pi / 2.0} 0.0 0.0" />  <!-- new offset -->
+        </xacro:unless>
       </collision>
       <xacro:cylinder_inertial radius="0.075" length="0.12" mass="${wrist_2_mass}">
@@ -221,8 +269,16 @@
       </visual>
       <collision>
-        <geometry>
-          <mesh filename="package://ur_description/meshes/ur10/collision/Wrist3.dae" scale="${scale}"/>
-        </geometry>
-         <origin xyz="0.0 -0.164 -1.427" rpy="${pi / 2.0} 0.0 0" />   <!-- new offset -->
+        <xacro:if value="${cylinders_collision}">
+          <geometry>
+            <cylinder length="0.147" radius="0.046" />
+          </geometry>
+          <origin xyz="0.0 0.017 0.0" rpy="${pi/2} 0.0 0.0" />
+        </xacro:if>
+        <xacro:unless value="${cylinders_collision}">
+          <geometry>
+            <mesh filename="package://ur_description/meshes/ur10/collision/Wrist3.dae" scale="${scale}"/>
+          </geometry>
+           <origin xyz="0.0 -0.164 -1.427" rpy="${pi / 2.0} 0.0 0" />   <!-- new offset -->
+        </xacro:unless>
       </collision>
       <xacro:cylinder_inertial radius="0.075" length="0.12" mass="${wrist_3_mass}">

File: ur_description/urdf/ur10_joint_limited_robot.urdf.xacro (robot description, xacro)
@@ -7,5 +7,5 @@
   <xacro:include filename="$(find ur_description)/urdf/ur10.urdf.xacro" />
   <!-- arm -->
-  <xacro:ur10_robot prefix=""
+  <xacro:ur10_robot prefix="" cylinders_collision="false"
                     j1_lwr_lmt="${-pi}" j1_upr_lmt="${pi}" j1_vel_lmt="2.16"
                     j2_lwr_lmt="${-pi}" j2_upr_lmt="${pi}" j2_vel_lmt="2.16"

File: ur_description/urdf/ur10_robot.urdf.xacro (robot description, xacro)
@@ -7,5 +7,5 @@
   <xacro:include filename="$(find ur_description)/urdf/ur10.urdf.xacro" />
   <!-- arm -->
-  <xacro:ur10_robot prefix=""
+  <xacro:ur10_robot prefix="" cylinders_collision="false"
                     j1_lwr_lmt="${-2.0*pi}" j1_upr_lmt="${2.0*pi}" j1_vel_lmt="2.16"
                     j2_lwr_lmt="${-2.0*pi}" j2_upr_lmt="${2.0*pi}" j2_vel_lmt="2.16"
