Commit message: Adding a few more cylinders.

File: ur_description/urdf/ur10.urdf.xacro (robot description, xacro)
@@ -64,18 +64,20 @@
         <material name="UR/Blue" />
       </visual>
-      <collision>
-        <xacro:if value="${cylinders_collision}">
+      <xacro:if value="${cylinders_collision}">
+        <collision>
           <geometry>
             <cylinder length="0.04" radius="0.10" />
           </geometry>
         <origin xyz="0.0 0.0 0.02" rpy="0.0 0.0 0.0" />
-        </xacro:if>
-        <xacro:unless value="${cylinders_collision}">
+        </collision>
+      </xacro:if>
+      <xacro:unless value="${cylinders_collision}">
+        <collision>
           <geometry>
             <mesh filename="package://ur_description/meshes/ur10/collision/Base.dae" scale="${scale}"/>
           </geometry>
           <origin xyz="0.0 0.0 0.0" rpy="${pi / 2.0} 0.0 0.0" />
-        </xacro:unless>
-      </collision>
+        </collision>
+      </xacro:unless>
       <xacro:cylinder_inertial radius="0.075" length="0.038" mass="${base_mass}">
         <origin xyz="0.0 0.0 0.0" rpy="0 0 0" />
@@ -98,18 +100,20 @@
         <material name="UR/Grey" />
       </visual>
-      <collision>
-        <xacro:if value="${cylinders_collision}">
+      <xacro:if value="${cylinders_collision}">
+        <collision>
           <geometry>
             <cylinder length="0.171" radius="0.08" />
           </geometry>
           <origin xyz="0.0 0.0 0.0" rpy="0.0 0.0 0.0" />
-        </xacro:if>
-        <xacro:unless value="${cylinders_collision}">
+        </collision>
+      </xacro:if>
+      <xacro:unless value="${cylinders_collision}">
+        <collision>
           <geometry>
             <mesh filename="package://ur_description/meshes/ur10/collision/Shoulder.dae" scale="${scale}"/>
           </geometry>
           <origin rpy="${pi / 2.0} 0.0 0.0" xyz="0.0 0.0 -0.127"/>   <!-- -0.127 ????  -->
-        </xacro:unless>
-      </collision>
+        </collision>
+      </xacro:unless>
       <xacro:cylinder_inertial radius="0.075" length="0.178" mass="${shoulder_mass}">
         <origin xyz="0.0 0.0 0.0" rpy="0 0 0" />
@@ -132,18 +136,26 @@
         <material name="UR/Blue" />
       </visual>
-      <collision>
-        <xacro:if value="${cylinders_collision}">
-          <geometry>
-            <cylinder length="${-ur10_a2+0.15}" radius="0.058" />
+      <xacro:if value="${cylinders_collision}">
+        <collision>
+          <geometry>
+            <cylinder length="${-ur10_a2+0.02}" radius="0.058" />
           </geometry>
           <origin xyz="0.0 -0.042 ${(-ur10_a2+0.15)/2-0.08}" rpy="0.0 0.0 0.0" />
-        </xacro:if>
-        <xacro:unless value="${cylinders_collision}">
+        </collision>
+        <collision>
+          <geometry>
+            <cylinder length="0.24" radius="0.08" />
+          </geometry>
+          <origin xyz="0.0 -0.08 0.0" rpy="${pi/2} 0.0 0.0" />
+        </collision>
+      </xacro:if>
+      <xacro:unless value="${cylinders_collision}">
+        <collision>
           <geometry>
             <mesh filename="package://ur_description/meshes/ur10/collision/UpperArm.dae" scale="${scale}"/>
           </geometry>
           <origin xyz="0.0 -0.221 -0.127" rpy="${pi / 2.0} 0.0 0.0" />  <!-- new offset-->
-        </xacro:unless>
-      </collision>
+        </collision>
+      </xacro:unless>
       <xacro:cylinder_inertial radius="0.075" length="${-ur10_a2}" mass="${upper_arm_mass}">
         <origin xyz="0.0 0.0 ${-ur10_a2/2.0}" rpy="0 0 0" />
@@ -166,18 +178,26 @@
         <material name="UR/Grey" />
       </visual>
-      <collision>
-        <xacro:if value="${cylinders_collision}">
+      <xacro:if value="${cylinders_collision}">
+        <collision>
           <geometry>
             <cylinder length="${(-ur10_a3+0.05)}" radius="0.048" />
           </geometry>
           <origin xyz="0.0 0.0 ${(-ur10_a3+0.05)/2-0.06}" rpy="0.0 0.0 0.0" />
-        </xacro:if>
-        <xacro:unless value="${cylinders_collision}">
+        </collision>
+        <collision>
+          <geometry>
+            <cylinder length="0.26" radius="0.06" />
+          </geometry>
+          <origin xyz="0.0 0.064 0.0" rpy="${pi/2} 0.0 0.0" />
+        </collision>
+      </xacro:if>
+      <xacro:unless value="${cylinders_collision}">
+        <collision>
           <geometry>
             <mesh filename="package://ur_description/meshes/ur10/collision/Forearm.dae" scale="${scale}"/>
           </geometry>
           <origin xyz="0.0 -0.049 -0.739" rpy="${pi / 2.0} 0.0 0.0" />  <!-- new offset -->
-        </xacro:unless>
-      </collision>
+        </collision>
+      </xacro:unless>
       <xacro:cylinder_inertial radius="0.075" length="${-ur10_a3}" mass="${forearm_mass}">
         <origin xyz="0.0 0.0 ${-ur10_a3/2.0}" rpy="0 0 0" />
@@ -200,18 +220,20 @@
         <material name="UR/Blue" />
       </visual>
-      <collision>
-        <xacro:if value="${cylinders_collision}">
-          <geometry>
-            <cylinder length="0.12" radius="0.047" />
-          </geometry>
-          <origin xyz="0.0 0.01 0.0" rpy="${pi/2} 0.0 0.0" />
-        </xacro:if>
-        <xacro:unless value="${cylinders_collision}">
+      <xacro:if value="${cylinders_collision}">
+        <collision>
+          <geometry>
+            <cylinder length="0.16" radius="0.047" />
+          </geometry>
+          <origin xyz="0.0 0.025 0.0" rpy="${pi/2} 0.0 0.0" />
+        </collision>
+      </xacro:if>
+      <xacro:unless value="${cylinders_collision}">
+        <collision>
           <geometry>
             <mesh filename="package://ur_description/meshes/ur10/collision/Wrist1.dae" scale="${scale}"/>
           </geometry>
           <origin xyz="0.0 -0.049 -1.312" rpy="${pi / 2.0} 0 0.0" />  <!-- new offset -->
-        </xacro:unless>
-      </collision>
+        </collision>
+      </xacro:unless>
       <xacro:cylinder_inertial radius="0.075" length="0.12" mass="${wrist_1_mass}">
         <origin xyz="0.0 0.0 0.0" rpy="0 0 0" />
@@ -234,18 +256,20 @@
         <material name="UR/Grey" />
       </visual>
-      <collision>
-        <xacro:if value="${cylinders_collision}">
+      <xacro:if value="${cylinders_collision}">
+        <collision>
           <geometry>
             <cylinder length="0.18" radius="0.046" />
           </geometry>
           <origin xyz="0.0 0.0 0.032" rpy="0.0 0.0 0.0" />
-        </xacro:if>
-        <xacro:unless value="${cylinders_collision}">
+        </collision>
+      </xacro:if>
+      <xacro:unless value="${cylinders_collision}">
+        <collision>
           <geometry>
             <mesh filename="package://ur_description/meshes/ur10/collision/Wrist2.dae" scale="${scale}"/>
           </geometry>
           <origin xyz="0.0 -0.164 -1.312" rpy="${pi / 2.0} 0.0 0.0" />  <!-- new offset -->
-        </xacro:unless>
-      </collision>
+        </collision>
+      </xacro:unless>
       <xacro:cylinder_inertial radius="0.075" length="0.12" mass="${wrist_2_mass}">
         <origin xyz="0.0 0.0 0.0" rpy="0 0 0" />
@@ -268,18 +292,20 @@
         <material name="UR/Blue" />
       </visual>
-      <collision>
-        <xacro:if value="${cylinders_collision}">
+      <xacro:if value="${cylinders_collision}">
+        <collision>
           <geometry>
             <cylinder length="0.147" radius="0.046" />
           </geometry>
           <origin xyz="0.0 0.017 0.0" rpy="${pi/2} 0.0 0.0" />
-        </xacro:if>
-        <xacro:unless value="${cylinders_collision}">
+        </collision>
+      </xacro:if>
+      <xacro:unless value="${cylinders_collision}">
+        <collision>
           <geometry>
             <mesh filename="package://ur_description/meshes/ur10/collision/Wrist3.dae" scale="${scale}"/>
           </geometry>
            <origin xyz="0.0 -0.164 -1.427" rpy="${pi / 2.0} 0.0 0" />   <!-- new offset -->
-        </xacro:unless>
-      </collision>
+        </collision>
+      </xacro:unless>
       <xacro:cylinder_inertial radius="0.075" length="0.12" mass="${wrist_3_mass}">
         <origin xyz="0.0 0.0 0.0" rpy="0 0 0" />
